File: PCBs/Tacho_Bottom/Tacho_Bottom.kicad_pcb (KiCad board)
At the start: 2 copper layers, 59 x 59 mm, 13 parts, among them J1 AudioJack3_Switch, J2 Voltage In, U1 ESP32-WROOM-32, U2 AMS1117-5.0, U3 AMS1117-3.3, U4 UDA1334ATS

Commit message: new Version
new Version
Parts:
- added C2: 0.1uF, Capacitor_SMD:C_0603_1608Metric_Pad1.08x0.95mm_HandSolder, B.Cu at (161.8, 72.1)
- added D1: LED_Small, LED_SMD:LED_1206_3216Metric_Pad1.42x1.75mm_HandSolder, F.Cu at (202.8, 101.4)
- added D2: 5V1, Diode_SMD:D_SOD-123, F.Cu at (207.3, 89.1)
- added J3: Conn_Coaxial, Connector_Coaxial:U.FL_Molex_MCRF_73412-0110_Vertical, F.Cu at (151.9, 123.1)
- added L1: 22uH, Inductor_SMD:L_12x12mm_H8mm, F.Cu at (192.4, 94.6)
- added R1: 22R, Resistor_SMD:R_0603_1608Metric_Pad0.98x0.95mm_HandSolder, F.Cu at (211.0, 92.1)
- added R2: 1k, Resistor_SMD:R_0603_1608Metric_Pad0.98x0.95mm_HandSolder, F.Cu at (206.6, 92.1)
- J1: value AudioJack3_Switch -> DISPLAY_Kilometer; footprint Connector_Audio:Jack_3.5mm_PJ311_Horizontal -> Connector_PinHeader_2.54mm:PinHeader_1x04_P2.54mm_Vertical
- U4: value UDA1334ATS -> NEO-8Q; footprint Package_SO:SSOP-16_4.4x5.2mm_P0.65mm -> RF_GPS:ublox_NEO; moved to B.Cu
- moved J1 56.1 mm to (202.1, 89.8), turned to 0 degrees
- moved U4 6.04 mm to (171.7, 84.8), turned to 180 degrees
Connections:
- J1 pad 1: (no net) -> unconnected-(J1-Pad1)
- J1 pad 2: (no net) -> unconnected-(J1-Pad2)
- J1 pad 3: (no net) -> unconnected-(J1-Pad3)
- J1 pad 4: (no net) -> unconnected-(J1-Pad4)
- U1 pad 24: unconnected-(U1-Pad24) -> /RDX0
- U1 pad 27: unconnected-(U1-Pad27) -> /RDX1
- U1 pad 28: unconnected-(U1-Pad28) -> /TDX1
- U1 pad 34: unconnected-(U1-Pad34) -> /RDX0
- U1 pad 35: unconnected-(U1-Pad35) -> /TDX0
- U4 pad 11: GND -> Net-(L1-Pad1)
- U4 pad 12: unconnected-(U4-Pad12) -> GND
- U4 pad 13: unconnected-(U4-Pad13) -> GND
- U4 pad 15: GND -> unconnected-(U4-Pad15)
- U4 pad 3: unconnected-(U4-Pad3) -> Net-(R2-Pad2)
- U4 pad 5: GND -> unconnected-(U4-Pad5)
- U4 pad 6: GND -> unconnected-(U4-Pad6)
- U4 pad 8: GND -> /RST-Neo
- U4 pad 9: unconnected-(U4-Pad9) -> /RST-Neo
