File: PCBs/Tacho_Bottom/Tacho_Bottom.kicad_sch (KiCad schematic)
At the start: 12 parts, among them J2 Voltage In, U1 ESP32-WROOM-32, U2 AMS1117-5.0, U3 AMS1117-3.3

Commit message: new Version
new Version
Parts:
- removed J?: AudioJack3_Switch, symbol Connector:AudioJack3_Switch
- removed U?: UDA1334ATS, Package_SO:SSOP-16_4.4x5.2mm_P0.65mm, symbol Audio:UDA1334ATS
- added C2: 0.1uF, Capacitor_SMD:C_0603_1608Metric_Pad1.08x0.95mm_HandSolder, symbol Device:C_Small
- added D1: LED_Small, LED_SMD:LED_1206_3216Metric_Pad1.42x1.75mm_HandSolder, symbol Device:LED_Small
- added D2: 5V1, Diode_SMD:D_SOD-123, symbol Device:D_Zener
- added J1: DISPLAY_Kilometer, Connector_PinHeader_2.54mm:PinHeader_1x04_P2.54mm_Vertical, symbol Connector:Conn_01x04_Female
- added J3: Conn_Coaxial, Connector_Coaxial:U.FL_Molex_MCRF_73412-0110_Vertical, symbol Connector:Conn_Coaxial
- added L1: 22uH, Inductor_SMD:L_12x12mm_H8mm, symbol Device:L
- added R1: 22R, Resistor_SMD:R_0603_1608Metric_Pad0.98x0.95mm_HandSolder, symbol Device:R_Small
- added R2: 1k, Resistor_SMD:R_0603_1608Metric_Pad0.98x0.95mm_HandSolder, symbol Device:R_Small
- added U4: NEO-8Q, RF_GPS:ublox_NEO, symbol RF_GPS:NEO-8Q
- added U5: CP2102N-Axx-xQFN20, Package_DFN_QFN:SiliconLabs_QFN-20-1EP_3x3mm_P0.5mm, symbol Interface_USB:CP2102N-Axx-xQFN20
Connections:
- net +3.3V: now also C2.1, U4.23 (VCC)
- net GND: now also C2.2, D1.1 (K), J3.2 (Ext), U4.10 (GND), U4.12 (GND), U4.13 (GND), U4.24 (GND), U4.7 (VDD_USB), U5.12 (GND), U5.21 (GND), U5.3 (GND)
- net RDX0: now reaches U1.24 (IO2)
- net RDX0: now also U1.34 (RXD0/IO3), U5.17 (RXD)
- net RDX1: now reaches U1.27 (IO16)
- net RDX1: now also U4.21 (RXD/SPI_MOSI)
- net TDX1: now reaches U1.28 (IO17)
- net TDX1: now also U4.20 (TXD/SPI_MISO)
- net TDX0: now reaches U1.35 (TXD0/IO1)
- net TDX0: now also U5.18 (TXD)
- new net: D1.2 (A), R2.1
- new net: R2.2, U4.3 (TIMEPULSE)
- new net: J3.1 (In), L1.1, U4.11 (RF_IN)
- new net: L1.2, R1.2
- new net RST-Neo: R1.1, U4.8 (~{RESET}), U4.9 (VCC_RF)
- new net SCL2: U4.19 (SCL/SPI_CLK)
- new net SDA2: U4.18 (SDA/~{SPI_CS})
